Commit message: ins 완성 테스트전

File: gazebo_dwa/husky_customization/husky_custom_description/urdf/custom_description_ouster_gps.urdf.xacro (robot description, xacro)
@@ -24,9 +24,9 @@
   <xacro:include filename="$(find husky_description)/urdf/husky.urdf.xacro" />
   <!-- Insert customization below, sample provided: -->
-  <!-- 2) OS1-32 LiDAR 모델 포함 -->
+  <!-- 2) OS1-64 LiDAR 모델 포함 -->
   <xacro:include filename="$(find ouster_description)/urdf/OS1-32.urdf.xacro"/>
   <xacro:OS1-32
-    parent="top_plate_link"
-    name="os_sensor"
+    parent="top_chassis_link"
+    name="ouster"
     topic_points="/ouster/points"
     topic_imu="/ouster/imu"
@@ -37,5 +37,5 @@
     max_range="50.0"
     noise="0.008"
-    lidar_link="os_lidar"
+    lidar_link="os_sensor"
     imu_link="os_imu"
     vfov_min="-.26"
@@ -45,6 +45,6 @@
    <!-- GPS 추가-->
   <!-- GPS 센서 포함 -->
-  <!-- <xacro:include filename="$(find husky_custom_description)/urdf/gps_sensor.urdf.xacro"/> -->
+  <xacro:include filename="$(find husky_custom_description)/urdf/gps_sensor.urdf.xacro"/>
   <!-- Gazebo 플러그인 포함 -->
-  <!-- <xacro:include filename="$(find husky_custom_gazebo)/urdf/custom_description.gazebo.xacro"/> -->
+  <xacro:include filename="$(find husky_custom_gazebo)/urdf/custom_description.gazebo.xacro"/>
 </robot>

File: gazebo_dwa/husky_customization/husky_custom_description/urdf/gps_sensor.urdf.xacro (robot description, xacro)
@@ -2,5 +2,5 @@
 <robot xmlns:xacro="http://www.ros.org/wiki/xacro">
   <!-- GPS Link -->
-  <link name="gps_link">
+  <link name="gps">
     <inertial>
       <mass value="0.001"/>
@@ -27,5 +27,5 @@
     <origin xyz="0.0 0.0 0.1" rpy="0 0 0"/>
     <parent link="base_link"/>
-    <child link="gps_link"/>
+    <child link="gps"/>
   </joint>
 </robot>

File: gazebo_dwa/husky_customization/husky_custom_gazebo/urdf/custom_description.gazebo.xacro (robot description, xacro)
@@ -33,15 +33,15 @@
   <!-- <xacro:husky_robot_gazebo /> -->
   <gazebo>
-    <plugin name="gps_sim" filename="libhector_gazebo_ros_gps.so">
+    <plugin name="gps" filename="libhector_gazebo_ros_gps.so">
       <robotNamespace>/</robotNamespace>
       <updateRate>10.0</updateRate>
       <bodyName>base_link</bodyName>
-      <frameId>gps_link</frameId>
-      <topicName>/gps/fix</topicName>
-      <velocityTopicName>/gps/fix_velocity</velocityTopicName>
-      <!-- 월드 좌표와 완전히 일치 -->
-      <referenceLatitude>0.0</referenceLatitude>
-      <referenceLongitude>0.0</referenceLongitude>
-      <referenceAltitude>0.0</referenceAltitude>
+      <frameId>gps</frameId>
+      <topicName>/ublox/fix</topicName>
+      <velocityTopicName>/ublox/fix_velocity</velocityTopicName>
+      <!-- 월드 좌표와 완전히 일치 (서울, 대한민국) -->
+      <referenceLatitude>37.5665</referenceLatitude>
+      <referenceLongitude>126.9780</referenceLongitude>
+      <referenceAltitude>38.0</referenceAltitude>
       <referenceHeading>0.0</referenceHeading>
       <!-- 매우 정밀한 시뮬레이션 설정 -->

File: gazebo_dwa/ouster_description/urdf/OS1-32.urdf.xacro (robot description, xacro)
@@ -111,4 +111,5 @@
       <updateRate>100.0</updateRate>
       <bodyName>${imu_link}</bodyName>
+      <frameId>${imu_link}</frameId>
       <topicName>${topic_imu}</topicName>
       <accelDrift>0.005 0.005 0.005</accelDrift>
@@ -118,4 +119,7 @@
       <headingDrift>0.005</headingDrift>
       <headingGaussianNoise>0.005</headingGaussianNoise>
+      <!-- Disable orientation output (real Ouster IMU doesn't provide orientation) -->
+      <rpyOffsets>0 0 0</rpyOffsets>
+      <gaussianNoise>0 0 0</gaussianNoise>
     </plugin>
   </gazebo>
